Commit message: update 3D models

File: fwdis/urdf/base/base.urdf.xacro (robot description, xacro)
@@ -10,17 +10,17 @@
     <link name="base_link">
       <visual>
-        <origin xyz="0.200 -0.630 0.060" rpy="${M_PI/2} 0 ${M_PI/2}"/>
+        <origin xyz="0 0 0" rpy="${M_PI/2} 0 ${M_PI/2}"/>
         <geometry>
-          <mesh filename="package://four_wheel_drive_independent_steering/meshes/STL/base.stl" scale="0.001 0.001 0.001"/>
+          <mesh filename="package://four_wheel_drive_independent_steering/meshes/STL/base2.stl" scale="0.001 0.001 0.001"/>
         </geometry>
       </visual>
       <collision>
-        <origin xyz="0.200 -0.630 0.060" rpy="${M_PI/2} 0 ${M_PI/2}"/>
+        <origin xyz="0 0 0" rpy="${M_PI/2} 0 ${M_PI/2}"/>
         <geometry>
-          <mesh filename="package://four_wheel_drive_independent_steering/meshes/STL/base.stl" scale="0.001 0.001 0.001"/>
+          <mesh filename="package://four_wheel_drive_independent_steering/meshes/STL/base2.stl" scale="0.001 0.001 0.001"/>
         </geometry>
       </collision>
       <inertial>
-        <origin xyz="0.200 -0.630 0.060" rpy="${M_PI/2} 0 ${M_PI/2}"/>
+        <origin xyz="0 0 0" rpy="${M_PI/2} 0 ${M_PI/2}"/>
         <box_inertial mass="5.0" height="0.5" width="0.5" depth="0.5"/>
         <mass value="43.24"/>

File: fwdis/urdf/steering/steering.urdf.xacro (robot description, xacro)
@@ -15,6 +15,7 @@
     <link name="${prefix}_steering_link">
       <visual>
+        <origin xyz="0 0 0" rpy="${M_PI/2} 0 ${M_PI/2}"/>
         <geometry>
-          <cylinder radius="${steering_radius}" length="${steering_width}"/>
+          <mesh filename="package://four_wheel_drive_independent_steering/meshes/STL/steering.stl" scale="0.001 0.001 0.001"/>
         </geometry>
       </visual>

File: fwdis/urdf/wheel/wheel.urdf.xacro (robot description, xacro)
@@ -2,7 +2,7 @@
 <robot xmlns:xacro="http://ros.org/wiki/xacro">
   <xacro:include filename="$(find four_wheel_drive_independent_steering)/urdf/common.xacro"/>
-  <property name="wheel_radius" value="0.075"/>
+  <property name="wheel_radius" value="0.100"/>
   <property name="wheel_width" value="0.030"/>
-  <property name="wheel_mass" value="2.0"/>
+  <property name="wheel_mass" value="1.0"/>
   <xacro:macro name="wheel" params="prefix parent *joint_origin *joint_axis">
     <joint name="${prefix}_wheel_joint" type="continuous">
@@ -15,10 +15,11 @@
     <link name="${prefix}_wheel_link">
       <visual>
+        <origin xyz="0 0.013208 0" rpy="${M_PI/2} 0 ${M_PI/2}"/>
         <geometry>
-          <cylinder radius="${wheel_radius}" length="${wheel_width}"/>
+          <mesh filename="package://four_wheel_drive_independent_steering/meshes/STL/wheel2.stl" scale="0.001 0.001 0.001"/>
         </geometry>
       </visual>
       <collision>
-        <origin xyz="0 0 0" rpy="0 0 0"/>
+        <origin xyz="0 0 0" rpy="${M_PI/2} 0 0"/>
         <geometry>
           <cylinder radius="${wheel_radius}" length="${wheel_width}"/>
@@ -26,5 +27,5 @@
       </collision>
       <inertial>
-        <origin xyz="0 0 0" rpy="0 0 0"/>
+        <origin xyz="0 0 0" rpy="${M_PI/2} 0 0"/>
         <cylinder_inertial mass="${wheel_mass}"
           radius="${wheel_radius}" length="${wheel_width}"/>
